File: PCB/Fuente.sch (KiCad schematic (older format))
At the start: 124 parts, among them P1 CONN_2, P10 CONN_2, P11 CONN_2, P12 CONN_2, P13 CONN_2, P14 CONN_2, P15 CONN_2, P16 CONN_2, P17 CONN_2, P18 CONN_2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

Commit message: Guarder
Parts:
- removed JP3, JP4, JP5: JUMPER, ~, symbol JUMPER
- gave numbers to parts that had none: 1
Connections:
- wire segments 526 -> 518
Other:
- moved on the sheet: P19, P20
